Commit message: add map server and a star node

File: description/camera.xacro (robot description, xacro)
@@ -4,10 +4,10 @@
         <parent link="chassis" />
         <child link="camera_link" />
-        <origin xyz="0.276 0 0.4" rpy="0 0 0" />
+        <origin xyz="0.276 0 0.7" rpy="0 0 0" />
     </joint>
     <link name="camera_link">
         <visual>
             <geometry>
-                <box size="0.010 0.03 0.03" />
+                <box size="0.025 0.09 0.025" />
             </geometry>
             <material name="black" />

File: description/robot.urdf.xacro (robot description, xacro)
@@ -10,6 +10,6 @@
         <xacro:include filename="gazebo_control.xacro" />
     </xacro:unless>
-    <!-- <xacro:include filename="lidar.xacro" /> -->
-    <xacro:include filename="camera.xacro" />
+    <xacro:include filename="lidar.xacro" />
+    <!-- <xacro:include filename="camera.xacro" /> -->
     <!-- <xacro:include filename="depth_camera.xacro" /> -->
     <xacro:include filename="face.xacro" />
